Commit message: change_lidar_color

File: my_robot_description/urdf/my_robot.urdf.xacro (robot description, xacro)
@@ -15,5 +15,5 @@
       		<xacro:box_inertial mass="1." sx="0.5" sy="0.25" sz="0.25">
 				<origin xyz="0 0 0" rpy="0 0 0"/>
-			</xacro:box_inertial>
+		</xacro:box_inertial>
 	</link>
 	<link name="lidar">
@@ -30,6 +30,9 @@
     		<xacro:cylinder_inertial mass="0.05" r="0.1" l="0.05">
 				<origin rpy="0 0 0" xyz="0 0 0"/>
-			</xacro:cylinder_inertial>
-	</link>
+		</xacro:cylinder_inertial>
+	</link>
+	<gazebo reference="lidar">
+		<material>Gazebo/Green</material>
+	</gazebo>
 	<link name="rightwheel">
 		<visual>
@@ -177,5 +180,5 @@
 		<material>Gazebo/FlatBlack</material>
 	</gazebo>
-			<gazebo reference="bras_droit">
+	<gazebo reference="bras_droit">
 		<mu1>1.2</mu1>
 		<mu2>1.2</mu2>

Commit message: controle_pinces

File: my_robot_description/urdf/my_robot.urdf.xacro (robot description, xacro)
@@ -12,21 +12,21 @@
            		<box size="0.5 0.25 0.25"/>
         	</geometry>
-      		</collision>
-      		<xacro:box_inertial mass="1." sx="0.5" sy="0.25" sz="0.25">
-				<origin xyz="0 0 0" rpy="0 0 0"/>
+  		</collision>
+  		<xacro:box_inertial mass="1." sx="0.5" sy="0.25" sz="0.25">
+			<origin xyz="0 0 0" rpy="0 0 0"/>
 		</xacro:box_inertial>
 	</link>
 	<link name="lidar">
-       		<visual>
-         		<geometry>
+   		<visual>
+     		<geometry>
 				<cylinder length="0.05" radius="0.1"/>
-         		</geometry>
-       		</visual>
-		<collision>
-  			<geometry>
-           			<cylinder length="0.05" radius="0.1"/>
-        	</geometry>
-      		</collision>
-    		<xacro:cylinder_inertial mass="0.05" r="0.1" l="0.05">
+     		</geometry>
+   		</visual>
+		<collision>
+  			<geometry>
+       			<cylinder length="0.05" radius="0.1"/>
+        	</geometry>
+  		</collision>
+		<xacro:cylinder_inertial mass="0.05" r="0.1" l="0.05">
 				<origin rpy="0 0 0" xyz="0 0 0"/>
 		</xacro:cylinder_inertial>
@@ -43,7 +43,7 @@
 		<collision>
   			<geometry>
-           			<cylinder length="0.05" radius="0.1"/>
-        	</geometry>
-      		</collision>
+       			<cylinder length="0.05" radius="0.1"/>
+        	</geometry>
+  		</collision>
     	<xacro:cylinder_inertial mass="0.3" r="0.1" l="0.05">
 			<origin rpy="0 0 0" xyz="0 0 0"/>
@@ -60,14 +60,14 @@
 	</gazebo>
 	<link name="leftwheel">
-       		<visual>
-         		<geometry>
+   		<visual>
+     		<geometry>
 				<cylinder length="0.05" radius="0.1"/>
-         		</geometry>
-       		</visual>
-		<collision>
-  			<geometry>
-           			<cylinder length="0.05" radius="0.1"/>
-        	</geometry>
-      		</collision>
+     		</geometry>
+   		</visual>
+		<collision>
+  			<geometry>
+       			<cylinder length="0.05" radius="0.1"/>
+        	</geometry>
+  		</collision>
     	<xacro:cylinder_inertial mass="0.3" r="0.1" l="0.05">
 			<origin rpy="0 0 0" xyz="0 0 0"/>
@@ -84,14 +84,14 @@
 	</gazebo>
 	<link name="crazywheel">
-       		<visual>
-         		<geometry>
+   		<visual>
+     		<geometry>
 				<sphere radius="0.05"/>
-         		</geometry>
-       		</visual>
-		<collision>
-  			<geometry>
-           			<sphere radius="0.05"/>
-        	</geometry>
-      		</collision>
+     		</geometry>
+   		</visual>
+		<collision>
+  			<geometry>
+       			<sphere radius="0.05"/>
+        	</geometry>
+  		</collision>
     	<xacro:sphere_inertial mass="0.05" r="0.05">
 			<origin rpy="0 0 0" xyz="0 0 0"/>
@@ -124,27 +124,27 @@
 			</xacro:box_inertial>
 	</link>
-		<link name="bras_gauche">
+	<link name="bras_gauche">
        	<visual>
        		<origin xyz = "0.29 0 0"/>
-         		<geometry>
-							<box size="0.60 0.05 0.05"/>
-         		</geometry>
-       		</visual>
+     		<geometry>
+				<box size="0.60 0.05 0.05"/>
+     		</geometry>
+   		</visual>
 		<collision>
 			<origin xyz = "0.29 0 0"/>
   			<geometry>
-           			<box size="0.60 0.05 0.05"/>
-        	</geometry>
-      		</collision>
+       			<box size="0.60 0.05 0.05"/>
+        	</geometry>
+  		</collision>
     	<xacro:box_inertial mass="0.1" sx="0.2" sy="0.05" sz="0.05">
-				<origin xyz="0 0 0" rpy="0 0 0"/>
-			</xacro:box_inertial>
-	</link>
-			<link name="boule_gauche">
+			<origin xyz="0 0 0" rpy="0 0 0"/>
+		</xacro:box_inertial>
+	</link>
+	<link name="boule_gauche">
        	<visual>
-         		<geometry>
-							<sphere radius="0.05"/>
-         		</geometry>
-       		</visual>
+     		<geometry>
+				<sphere radius="0.05"/>
+     		</geometry>
+   		</visual>
 		<collision>
   			<geometry>
@@ -153,23 +153,23 @@
       		</collision>
     	<xacro:sphere_inertial mass="0.05" r="0.05">
-				<origin xyz="0 0 0" rpy="0 0 0"/>
-			</xacro:sphere_inertial>
-	</link>
-			<link name="boule_droite">
+			<origin xyz="0 0 0" rpy="0 0 0"/>
+		</xacro:sphere_inertial>
+	</link>
+	<link name="boule_droite">
        	<visual>
-         		<geometry>
-							<sphere radius="0.05"/>
-         		</geometry>
-       		</visual>
+     		<geometry>
+				<sphere radius="0.05"/>
+     		</geometry>
+       	</visual>
 		<collision>
   			<geometry>
            		<sphere radius="0.05"/>
         	</geometry>
-      		</collision>
+      	</collision>
     	<xacro:sphere_inertial mass="0.05" r="0.05">
 			<origin rpy="0 0 0" xyz="0 0 0"/>
 		</xacro:sphere_inertial>
 	</link>
-		<gazebo reference="bras_gauche">
+	<gazebo reference="bras_gauche">
 		<mu1>1.2</mu1>
 		<mu2>1.2</mu2>
@@ -224,7 +224,7 @@
 		<axis xyz="0 0 1" />
 	</joint>
-		<joint name="bras_gauche_to_boule" type="fixed">
-     		<parent link="bras_gauche"/>
-     		<child link="boule_gauche"/>
+	<joint name="bras_gauche_to_boule" type="fixed">
+	     	<parent link="bras_gauche"/>
+	     	<child link="boule_gauche"/>
 		<origin rpy="0 0 0" xyz="0.61 0 0"/>
 	</joint>
@@ -237,6 +237,10 @@
 	<gazebo>
 		<plugin name='diff_drive' filename='libgazebo_ros_diff_drive.so'>
-			<!-- wheels -->
-			<command_topic>cmd_vel_0</command_topic>
+			<ros>
+				<!-- Remap default topics -->
+	          <argument>cmd_vel:=cmd_roues</argument>
+	          <argument>odom:=odom_roues</argument>
+	        </ros>
+        <!-- wheels -->
 			<left_joint>base_to_leftwheel</left_joint>
 			<right_joint>base_to_rightwheel</right_joint>
@@ -257,11 +261,10 @@
 	<gazebo>
 		<plugin name='diff_drive_pince' filename='libgazebo_ros_diff_drive.so'>
-			<!-- wheels -->
-			  <ros>
-          <!-- Set namespace -->
-          <!-- Remap default topics -->
-          <argument>cmd_vel:=cmd_demo</argument>
-          <argument>odom:=odom_demo</argument>
-        </ros>
+			<ros>
+	          <!-- Remap default topics -->
+	          <argument>cmd_vel:=cmd_pince</argument>
+	          <argument>odom:=odom_pince</argument>
+	        </ros>
+        	<!-- wheels -->
 			<left_joint>base_to_bras_droit</left_joint>
 			<right_joint>base_to_bras_gauche</right_joint>

Commit message: publishers pour liaison

File: my_robot_description/urdf/my_robot.urdf.xacro (robot description, xacro)
@@ -156,4 +156,13 @@
 		</xacro:sphere_inertial>
 	</link>
+	<gazebo reference="boule_gauche">
+		<mu1>5</mu1>
+		<mu2>5</mu2>
+		<kp>500000.0</kp>
+		<kd>10.0</kd>
+		<minDepth>0.001</minDepth>
+		<maxVel>0.1</maxVel>
+		<material>Gazebo/FlatBlack</material>
+	</gazebo>
 	<link name="boule_droite">
        	<visual>
@@ -171,4 +180,13 @@
 		</xacro:sphere_inertial>
 	</link>
+	<gazebo reference="boule_droite">
+		<mu1>5</mu1>
+		<mu2>5</mu2>
+		<kp>500000.0</kp>
+		<kd>10.0</kd>
+		<minDepth>0.001</minDepth>
+		<maxVel>0.1</maxVel>
+		<material>Gazebo/FlatBlack</material>
+	</gazebo>
 	<gazebo reference="bras_gauche">
 		<mu1>1.2</mu1>

Commit message: adapt_controller

File: my_robot_description/urdf/my_robot.urdf.xacro (robot description, xacro)
@@ -111,5 +111,5 @@
        		<origin xyz = "0.29 0 0"/>
          		<geometry>
-							<box size="0.60 0.05 0.05"/>
+							<box size="0.60 0.05 0.2"/>
          		</geometry>
        		</visual>
@@ -117,5 +117,5 @@
 			<origin xyz = "0.29 0 0"/>
   			<geometry>
-           			<box size="0.60 0.05 0.05"/>
+           			<box size="0.60 0.05 0.2"/>
         	</geometry>
       		</collision>
@@ -128,5 +128,5 @@
        		<origin xyz = "0.29 0 0"/>
      		<geometry>
-				<box size="0.60 0.05 0.05"/>
+				<box size="0.60 0.05 0.2"/>
      		</geometry>
    		</visual>
@@ -134,5 +134,5 @@
 			<origin xyz = "0.29 0 0"/>
   			<geometry>
-       			<box size="0.60 0.05 0.05"/>
+       			<box size="0.60 0.05 0.2"/>
         	</geometry>
   		</collision>
@@ -144,10 +144,10 @@
        	<visual>
      		<geometry>
-				<sphere radius="0.05"/>
-     		</geometry>
-   		</visual>
-		<collision>
-  			<geometry>
-           		<sphere radius="0.05"/>
+				<sphere radius="0.07"/>
+     		</geometry>
+   		</visual>
+		<collision>
+  			<geometry>
+           		<sphere radius="0.07"/>
         	</geometry>
       		</collision>
@@ -157,6 +157,6 @@
 	</link>
 	<gazebo reference="boule_gauche">
-		<mu1>5</mu1>
-		<mu2>5</mu2>
+		<mu1>0.1</mu1>
+		<mu2>0.1</mu2>
 		<kp>500000.0</kp>
 		<kd>10.0</kd>
@@ -168,10 +168,10 @@
        	<visual>
      		<geometry>
-				<sphere radius="0.05"/>
+				<sphere radius="0.07"/>
      		</geometry>
        	</visual>
 		<collision>
   			<geometry>
-           		<sphere radius="0.05"/>
+           		<sphere radius="0.07"/>
         	</geometry>
       	</collision>
@@ -181,6 +181,6 @@
 	</link>
 	<gazebo reference="boule_droite">
-		<mu1>5</mu1>
-		<mu2>5</mu2>
+		<mu1>0.1</mu1>
+		<mu2>0.1</mu2>
 		<kp>500000.0</kp>
 		<kd>10.0</kd>
@@ -190,6 +190,6 @@
 	</gazebo>
 	<gazebo reference="bras_gauche">
-		<mu1>1.2</mu1>
-		<mu2>1.2</mu2>
+		<mu1>0.1</mu1>
+		<mu2>0.1</mu2>
 		<kp>500000.0</kp>
 		<kd>10.0</kd>
@@ -199,6 +199,6 @@
 	</gazebo>
 	<gazebo reference="bras_droit">
-		<mu1>1.2</mu1>
-		<mu2>1.2</mu2>
+		<mu1>0.1</mu1>
+		<mu2>0.1</mu2>
 		<kp>500000.0</kp>
 		<kd>10.0</kd>
@@ -233,5 +233,5 @@
      		<parent link="base_link"/>
      		<child link="bras_droit"/>
-		<origin rpy="0 0 -0.2" xyz="0.25 -0.07 -0.1"/>
+		<origin rpy="0 0 -0.2" xyz="0.25 -0.07 -0.06"/>
 		<axis xyz="0 0 1" />
 	</joint>
@@ -239,5 +239,5 @@
      		<parent link="base_link"/>
      		<child link="bras_gauche"/>
-		<origin rpy="0 0 0.2" xyz="0.25 0.07 -0.1"/>
+		<origin rpy="0 0 0.2" xyz="0.25 0.07 -0.06"/>
 		<axis xyz="0 0 1" />
 	</joint>
@@ -245,10 +245,10 @@
 	     	<parent link="bras_gauche"/>
 	     	<child link="boule_gauche"/>
-		<origin rpy="0 0 0" xyz="0.61 0 0"/>
+		<origin rpy="0 0 0" xyz="0.61 -0.02 -0.05"/>
 	</joint>
 	<joint name="bras_droite_to_boule" type="fixed">
      		<parent link="bras_droit"/>
      		<child link="boule_droite"/>
-		<origin rpy="0 0 0" xyz="0.61 0 0"/>
+		<origin rpy="0 0 0" xyz="0.61 0.02 -0.05"/>
 	</joint>
 	<!--> __________________________________________________________ </!-->
@@ -301,30 +301,3 @@
 		</plugin>
 	</gazebo>
-	<gazebo reference="lidar">
-		<sensor name="sensor_ray" type="ray">
-		<ray>
-			<scan>
-				<horizontal>
-					<samples>720</samples>
-					<resolution>1.0</resolution>
-					<min_angle>-1.57</min_angle>
-					<max_angle>1.57</max_angle>
-				</horizontal>
-			</scan>
-			<range>
-				<min>0.2</min>
-				<max>20.0</max>
-			</range>
-		</ray>
-		<always_on>true</always_on>
-		<update_rate>10</update_rate>
-		<visualize>true</visualize>
-		<plugin name="laserscan" filename="libgazebo_ros_ray_sensor.so">
-			<ros>
-				<remapping>~/out:=scan</remapping>
-			</ros>
-			<output_type>sensor_msgs/LaserScan</output_type>
-		</plugin>
-		</sensor>
-	</gazebo>
 </robot>

Commit message: vacuum

File: my_robot_description/urdf/my_robot.urdf.xacro (robot description, xacro)
@@ -211,4 +211,19 @@
 		<material>Gazebo/FlatBlack</material>
 	</gazebo>
+	<link name="vacuum_gripper">
+	    <gravity>0</gravity>
+	    <visual>
+	      <origin rpy="0 0 0" xyz="0 0 0"/>
+	      <geometry>
+		<cylinder radius="0.005" length="0.01"/>
+	      </geometry>
+	      <material name="transparent">
+		<color rgba="0 0 0 0"/>
+	      </material>
+	    </visual>
+      <xacro:sphere_inertial mass="0.05" r="0.05">
+      <origin rpy="0 0 0" xyz="0 0 0"/>
+    </xacro:sphere_inertial>
+	  </link>
 	<!--> __________________________________________________________ </!-->
 	<joint name="base_to_lidar" type="fixed">
@@ -256,4 +271,12 @@
 		<origin rpy="0 0 0" xyz="0.61 0.02 -0.05"/>
 	</joint>
+	    <joint name="gripper_joint" type="revolute">
+	      <axis xyz="1 0 0" />
+	      <parent link="base_link" />
+	      <child link="vacuum_gripper" />
+	      <origin rpy="0 1.5708 0" xyz="0.0 0.125 -0.1" />
+	      <limit effort="50" velocity="50" lower="0" upper="0" />
+	      <dynamics damping="0.0" friction="10"/>
+	    </joint>
 	<!--> __________________________________________________________ </!-->
 	<gazebo>
@@ -305,3 +328,10 @@
 		</plugin>
 	</gazebo>
+  <gazebo>
+      <plugin name="gazebo_ros_vacuum_gripper" filename="libgazebo_ros_vacuum_gripper.so">
+        <link_name>vacuum_gripper</link_name>
+  	<max_force>100000</max_force>
+  	<max_distance>10.0</max_distance>
+      </plugin>
+  </gazebo>
 </robot>

Commit message: mid day commit

File: my_robot_description/urdf/my_robot.urdf.xacro (robot description, xacro)
@@ -111,5 +111,5 @@
        		<origin xyz = "0.29 0 0"/>
          		<geometry>
-							<box size="0.60 0.05 0.2"/>
+				<box size="0.40 0.05 0.2"/>
          		</geometry>
        		</visual>
@@ -117,6 +117,6 @@
 			<origin xyz = "0.29 0 0"/>
   			<geometry>
-           			<box size="0.60 0.05 0.2"/>
-        	</geometry>
+           			<box size="0.40 0.05 0.2"/>
+        		</geometry>
       		</collision>
     	<xacro:box_inertial mass="0.1" sx="0.2" sy="0.05" sz="0.05">
@@ -128,5 +128,5 @@
        		<origin xyz = "0.29 0 0"/>
      		<geometry>
-				<box size="0.60 0.05 0.2"/>
+				<box size="0.40 0.05 0.2"/>
      		</geometry>
    		</visual>
@@ -134,5 +134,5 @@
 			<origin xyz = "0.29 0 0"/>
   			<geometry>
-       			<box size="0.60 0.05 0.2"/>
+       			<box size="0.40 0.05 0.2"/>
         	</geometry>
   		</collision>
@@ -252,5 +252,5 @@
      		<parent link="base_link"/>
      		<child link="bras_droit"/>
-		<origin rpy="0 0 -0.2" xyz="0.25 -0.07 -0.06"/>
+		<origin rpy="0 0 -0.2" xyz="0.15 -0.07 -0.06"/>
 		<axis xyz="0 0 1" />
 	</joint>
@@ -258,5 +258,5 @@
      		<parent link="base_link"/>
      		<child link="bras_gauche"/>
-		<origin rpy="0 0 0.2" xyz="0.25 0.07 -0.06"/>
+		<origin rpy="0 0 0.2" xyz="0.15 0.07 -0.06"/>
 		<axis xyz="0 0 1" />
 	</joint>
@@ -264,10 +264,10 @@
 	     	<parent link="bras_gauche"/>
 	     	<child link="boule_gauche"/>
-		<origin rpy="0 0 0" xyz="0.61 -0.02 -0.05"/>
+		<origin rpy="0 0 0" xyz="0.51 -0.02 -0.05"/>
 	</joint>
 	<joint name="bras_droite_to_boule" type="fixed">
      		<parent link="bras_droit"/>
      		<child link="boule_droite"/>
-		<origin rpy="0 0 0" xyz="0.61 0.02 -0.05"/>
+		<origin rpy="0 0 0" xyz="0.51 0.02 -0.05"/>
 	</joint>
 	    <joint name="gripper_joint" type="revolute">
