Commit message: almost working

File: my_robot_description/urdf/my_robot.urdf.xacro (robot description, xacro)
@@ -20,5 +20,5 @@
    		<visual>
      		<geometry>
-				<cylinder length="0.05" radius="0.1"/>
+			<cylinder length="0.05" radius="0.1"/>
      		</geometry>
    		</visual>
@@ -29,5 +29,5 @@
   		</collision>
 		<xacro:cylinder_inertial mass="0.05" r="0.1" l="0.05">
-				<origin rpy="0 0 0" xyz="0 0 0"/>
+			<origin rpy="0 0 0" xyz="0 0 0"/>
 		</xacro:cylinder_inertial>
 	</link>
@@ -38,13 +38,13 @@
 		<visual>
 			<geometry>
-         		<cylinder length="0.05" radius="0.1"/>
+         			<cylinder length="0.05" radius="0.1"/>
 			</geometry>
        	</visual>
 		<collision>
   			<geometry>
-       			<cylinder length="0.05" radius="0.1"/>
-        	</geometry>
-  		</collision>
-    	<xacro:cylinder_inertial mass="0.3" r="0.1" l="0.05">
+       				<cylinder length="0.05" radius="0.1"/>
+        		</geometry>
+  		</collision>
+    		<xacro:cylinder_inertial mass="0.3" r="0.1" l="0.05">
 			<origin rpy="0 0 0" xyz="0 0 0"/>
 		</xacro:cylinder_inertial>
@@ -62,16 +62,16 @@
    		<visual>
      		<geometry>
-				<cylinder length="0.05" radius="0.1"/>
-     		</geometry>
-   		</visual>
-		<collision>
-  			<geometry>
-       			<cylinder length="0.05" radius="0.1"/>
-        	</geometry>
-  		</collision>
-    	<xacro:cylinder_inertial mass="0.3" r="0.1" l="0.05">
+			<cylinder length="0.05" radius="0.1"/>
+     		</geometry>
+   		</visual>
+		<collision>
+  			<geometry>
+       				<cylinder length="0.05" radius="0.1"/>
+        		</geometry>
+  		</collision>
+    		<xacro:cylinder_inertial mass="0.3" r="0.1" l="0.05">
 			<origin rpy="0 0 0" xyz="0 0 0"/>
 		</xacro:cylinder_inertial>
-     </link>
+     	</link>
 	<gazebo reference="leftwheel">
 		<mu1>2.0</mu1>
@@ -86,13 +86,13 @@
    		<visual>
      		<geometry>
-				<sphere radius="0.05"/>
-     		</geometry>
-   		</visual>
-		<collision>
-  			<geometry>
-       			<sphere radius="0.05"/>
-        	</geometry>
-  		</collision>
-    	<xacro:sphere_inertial mass="0.05" r="0.05">
+			<sphere radius="0.05"/>
+     		</geometry>
+   		</visual>
+		<collision>
+  			<geometry>
+       				<sphere radius="0.05"/>
+        		</geometry>
+  		</collision>
+    		<xacro:sphere_inertial mass="0.05" r="0.05">
 			<origin rpy="0 0 0" xyz="0 0 0"/>
 		</xacro:sphere_inertial>
@@ -120,7 +120,7 @@
         		</geometry>
       		</collision>
-    	<xacro:box_inertial mass="0.1" sx="0.2" sy="0.05" sz="0.05">
-				<origin xyz="0 0 0" rpy="0 0 0"/>
-			</xacro:box_inertial>
+    		<xacro:box_inertial mass="0.1" sx="0.2" sy="0.05" sz="0.05">
+			<origin xyz="0 0 0" rpy="0 0 0"/>
+		</xacro:box_inertial>
 	</link>
 	<link name="bras_gauche">
@@ -128,14 +128,14 @@
        		<origin xyz = "0.29 0 0"/>
      		<geometry>
-				<box size="0.40 0.05 0.2"/>
+			<box size="0.40 0.05 0.2"/>
      		</geometry>
    		</visual>
 		<collision>
 			<origin xyz = "0.29 0 0"/>
-  			<geometry>
+  				<geometry>
        			<box size="0.40 0.05 0.2"/>
         	</geometry>
   		</collision>
-    	<xacro:box_inertial mass="0.1" sx="0.2" sy="0.05" sz="0.05">
+    		<xacro:box_inertial mass="0.1" sx="0.2" sy="0.05" sz="0.05">
 			<origin xyz="0 0 0" rpy="0 0 0"/>
 		</xacro:box_inertial>
@@ -144,5 +144,5 @@
        	<visual>
      		<geometry>
-				<sphere radius="0.07"/>
+			<sphere radius="0.07"/>
      		</geometry>
    		</visual>
@@ -152,10 +152,10 @@
         	</geometry>
       		</collision>
-    	<xacro:sphere_inertial mass="0.05" r="0.05">
+    		<xacro:sphere_inertial mass="0.05" r="0.05">
 			<origin xyz="0 0 0" rpy="0 0 0"/>
 		</xacro:sphere_inertial>
 	</link>
 	<gazebo reference="boule_gauche">
-   		 <selfCollide>true</selfCollide>
+   		<selfCollide>true</selfCollide>
 		<mu1>0.1</mu1>
 		<mu2>0.1</mu2>
@@ -167,20 +167,20 @@
 	</gazebo>
 	<link name="boule_droite">
-       	<visual>
-     		<geometry>
+       		<visual>
+     			<geometry>
 				<sphere radius="0.07"/>
-     		</geometry>
-       	</visual>
-		<collision>
-  			<geometry>
-           		<sphere radius="0.07"/>
-        	</geometry>
-      	</collision>
-    	<xacro:sphere_inertial mass="0.05" r="0.05">
+     			</geometry>
+       		</visual>
+		<collision>
+  			<geometry>
+           			<sphere radius="0.07"/>
+        		</geometry>
+      		</collision>
+    		<xacro:sphere_inertial mass="0.05" r="0.05">
 			<origin rpy="0 0 0" xyz="0 0 0"/>
 		</xacro:sphere_inertial>
 	</link>
 	<gazebo reference="boule_droite">
-    <selfCollide>true</selfCollide>
+    		<selfCollide>true</selfCollide>
 		<mu1>0.1</mu1>
 		<mu2>0.1</mu2>
@@ -192,5 +192,5 @@
 	</gazebo>
 	<gazebo reference="bras_gauche">
-    <selfCollide>true</selfCollide>
+    		<selfCollide>true</selfCollide>
 		<mu1>0.1</mu1>
 		<mu2>0.1</mu2>
@@ -202,5 +202,5 @@
 	</gazebo>
 	<gazebo reference="bras_droit">
-    <selfCollide>true</selfCollide>
+    		<selfCollide>true</selfCollide>
 		<mu1>0.1</mu1>
 		<mu2>0.1</mu2>
@@ -212,17 +212,17 @@
 	</gazebo>
 	<link name="vacuum_gripper">
-	    <gravity>0</gravity>
-	    <visual>
-	      <origin rpy="0 0 0" xyz="0 0 0"/>
-	      <geometry>
-		<cylinder radius="0.005" length="0.01"/>
-	      </geometry>
-	      <material name="transparent">
-		<color rgba="0 0 0 0"/>
-	      </material>
-	    </visual>
-      <xacro:sphere_inertial mass="0.05" r="0.05">
-      <origin rpy="0 0 0" xyz="0 0 0"/>
-    </xacro:sphere_inertial>
+		<gravity>0</gravity>
+	    	<visual>
+	    		<origin rpy="0 0 0" xyz="0 0 0"/>
+	      			<geometry>
+					<cylinder radius="0.005" length="0.01"/>
+	      			</geometry>
+	      		<material name="transparent">
+				<color rgba="0 0 0 0"/>
+	      		</material>
+	    	</visual>
+      		<xacro:sphere_inertial mass="0.05" r="0.05">
+      			<origin rpy="0 0 0" xyz="0 0 0"/>
+    		</xacro:sphere_inertial>
 	  </link>
 	<!--> __________________________________________________________ </!-->
@@ -247,5 +247,5 @@
      		<parent link="base_link"/>
      		<child link="crazywheel"/>
-     	<origin rpy="0 0 0" xyz="0.15 0 -0.125"/>
+     		<origin rpy="0 0 0" xyz="0.15 0 -0.125"/>
 	</joint>
 	<joint name="base_to_bras_droit" type="continuous">
@@ -271,5 +271,5 @@
 		<origin rpy="0 0 0" xyz="0.51 0.02 -0.05"/>
 	</joint>
-	    <joint name="gripper_joint" type="revolute">
+	<joint name="gripper_joint" type="revolute">
 	      <axis xyz="1 0 0" />
 	      <parent link="base_link" />
@@ -278,14 +278,13 @@
 	      <limit effort="50" velocity="50" lower="0" upper="0" />
 	      <dynamics damping="0.0" friction="10"/>
-	    </joint>
+	</joint>
 	<!--> __________________________________________________________ </!-->
 	<gazebo>
 		<plugin name='diff_drive' filename='libgazebo_ros_diff_drive.so'>
-			<ros>
-				<!-- Remap default topics -->
-	          <argument>cmd_vel:=cmd_roues</argument>
-	          <argument>odom:=odom_roues</argument>
-	        </ros>
-        <!-- wheels -->
+			<ros> <!-- Remap default topics -->
+	         		<argument>cmd_vel:=cmd_roues</argument>
+	          		<argument>odom:=odom_roues</argument>
+	        	</ros>
+        		<!-- wheels -->
 			<left_joint>base_to_leftwheel</left_joint>
 			<right_joint>base_to_rightwheel</right_joint>
@@ -306,10 +305,9 @@
 	<gazebo>
 		<plugin name='diff_drive_pince' filename='libgazebo_ros_diff_drive.so'>
-			<ros>
-	          <!-- Remap default topics -->
-	          <argument>cmd_vel:=cmd_pince</argument>
-	          <argument>odom:=odom_pince</argument>
-	        </ros>
-        	<!-- wheels -->
+			<ros> <!-- Remap default topics -->
+			  <argument>cmd_vel:=cmd_pince</argument>
+			  <argument>odom:=odom_pince</argument>
+			</ros>
+			<!-- wheels -->
 			<left_joint>base_to_bras_droit</left_joint>
 			<right_joint>base_to_bras_gauche</right_joint>
@@ -328,10 +326,10 @@
 		</plugin>
 	</gazebo>
-  <gazebo>
-      <plugin name="gazebo_ros_vacuum_gripper" filename="libgazebo_ros_vacuum_gripper.so">
-        <link_name>vacuum_gripper</link_name>
-  	<max_force>0.01</max_force>
-  	<max_distance>1.5</max_distance>
-      </plugin>
-  </gazebo>
+	<gazebo>
+		<plugin name="gazebo_ros_vacuum_gripper" filename="libgazebo_ros_vacuum_gripper.so">
+			<link_name>vacuum_gripper</link_name>
+	  		<max_force>0.01</max_force>
+	  		<max_distance>1.5</max_distance>
+	      	</plugin>
+	</gazebo>
 </robot>

Commit message: almost working fix

File: my_robot_description/urdf/my_robot.urdf.xacro (robot description, xacro)
@@ -252,5 +252,5 @@
      		<parent link="base_link"/>
      		<child link="bras_droit"/>
-		<origin rpy="0 0 -0.2" xyz="0.15 -0.07 -0.06"/>
+		<origin rpy="0 0 -0.2" xyz="0.15 -0.07 -0.05"/>
 		<axis xyz="0 0 1" />
 	</joint>
@@ -258,5 +258,5 @@
      		<parent link="base_link"/>
      		<child link="bras_gauche"/>
-		<origin rpy="0 0 0.2" xyz="0.15 0.07 -0.06"/>
+		<origin rpy="0 0 0.2" xyz="0.15 0.07 -0.05"/>
 		<axis xyz="0 0 1" />
 	</joint>
@@ -329,6 +329,6 @@
 		<plugin name="gazebo_ros_vacuum_gripper" filename="libgazebo_ros_vacuum_gripper.so">
 			<link_name>vacuum_gripper</link_name>
-	  		<max_force>0.01</max_force>
-	  		<max_distance>1.5</max_distance>
+	  		<max_force>0.5</max_force>
+	  		<max_distance>2.</max_distance>
 	      	</plugin>
 	</gazebo>
